Commit message: integration on sonar ready

File: ros_ws/src/base_packages/bluerov2/bluerov2_description/urdf/sensors.xacro (robot description, xacro)
@@ -34,3 +34,18 @@
     <origin xyz="0.2 0 0" rpy="0 0 0"/>
   </sensor_d435>
+  <xacro:bluerov2_sss namespace="$(arg namespace)" parent_link="$(arg namespace)/base_link" topic="sonar_" mass="0.1"
+                      update_rate="15" samples="100" fov="2.27" range_min="0.1"
+                      range_max="1000.0"
+                      range_stddev="0.27"
+                      mesh=""
+                      suffix="forward">
+          <inertia ixx="0.00001" ixy="0.0" ixz="0.0" iyy="0.00001" iyz="0.0" izz="0.00001" />
+          <origin xyz="0.2 0 -0.05" rpy="0 0 0"/>
+          <visual>
+            <origin xyz="0.2 0 -0.05" rpy="0 0 0"/>
+            <geometry>
+              <box size="0.1 0.1 0.1"/>
+            </geometry>
+          </visual>
+  </xacro:bluerov2_sss>
 </robot>
